Commit message: 升降台成功接入,且能控制高度

File: assets/bookarm_urdf/urdf/bookarm_urdf.urdf (robot description, URDF)
Before this commit: robot bookarm_urdf, 7 links, 6 joints
Joints:
- joint joint_pole: limit lower=-1.26 upper=1.94 effort=1 velocity=1 -> lower=-1.26 upper=2.36 effort=1 velocity=1

Commit message: 抓放全流程初步完成

File: assets/bookarm_urdf/urdf/bookarm_urdf.urdf (robot description, URDF)
Before this commit: robot bookarm_urdf, 7 links, 6 joints
Joints:
- joint joint1_base: limit lower=-3.14159 upper=3.14159 effort=1 velocity=1 -> lower=-6.283185307179586 upper=6.283185307179586 effort=1 velocity=1
